File: PCB/Keyboard65.kicad_pcb (KiCad board)
At the start: 2 copper layers, 320 x 110 mm, 132 parts, among them SW1 SW_Push, SW10 SW_Push, SW11 SW_Push, SW12 SW_Push, SW13 SW_Push, SW14 SW_Push, SW15 SW_Push, SW16 SW_Push, SW17 SW_Push, SW18 SW_Push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

Commit message: Update the silkscreen and the PCB files
Parts:
- added G***: LOGO, LOGO, F.Cu at (455.0, 156.0)
